File: pedal/pedal.kicad_sch (KiCad schematic)
At the start: 46 parts, among them J1 AudioJack3, J2 AudioJack3, J3 Micro SD, J4 USB_B_Micro, J5 Debug, U1 LP2985-1.8, U2 PCM3060, U3 TPS62172DSG, U5 STM32H750IBTx, Y1 25MHz

Commit message: Review TPS62172
Parts:
- removed R3: 100R, symbol Device:R
- added C30: 10uF, symbol Device:C
- added R3: 100k, symbol Device:R_Small
- C28: value 4.7uF -> 2.2uF
Connections:
- net +9V is gone; now on net +3V3: U3.2 (VIN), U3.3 (EN)
- net GNDD is gone; now on net +3V3: C1.1, C10.2, C11.2, C12.2, C13.2, C14.2, C15.2, C16.2, C17.2, C2.1, C21.2, C24.1, C25.1, C3.2, C4.2, C5.2, C6.2, C7.2, C8.2, C9.2, J4.5 (GND), QSPI.10 (GND), SDRAM.12 (GNDQ), SDRAM.28 (GND), SDRAM.41 (GND), SDRAM.46 (GNDQ), SDRAM.52 (GNDQ), SDRAM.54 (GND), SDRAM.6 (GNDQ), U2.8 (DGND), U5.102 (VSS), U5.113 (VSS), U5.126 (VSS), U5.135 (VSS), U5.14 (VSS), U5.148 (VSS), U5.158 (VSS), U5.22 (VSS), U5.48 (VSS), U5.61 (VSS), U5.71 (VSS), U5.90 (VSS)
- net +3V3: now also C26.2, C27.2, C28.2, U1.2 (GND), U3.1 (PGND), U3.4 (AGND), C30.1, C30.2, R3.1, R3.2
- net GNDA: now also U3.9 (PAD); no longer C26.2, C27.2, C28.2, U1.2 (GND)
- net SAI1_FS: now reaches U5.3 (PE4)
- net SAI1_FS: now also U2.4 (LRCK1)
- net SAI1_SCK: now reaches U5.4 (PE5)
- net SAI1_SCK: now also U2.5 (BCK1)

Commit message: Update QSPI flash
Parts:
- added C31: 100nF, symbol Device:C
- added C32: 10uF, symbol Device:C
- added U4: TL072, symbol Amplifier_Operational:TL072
- added U6: RC4580, symbol Amplifier_Operational:RC4580
Connections:
- net +1V8: now also QSPI.2 (VCC), C31.1, C32.1
- net GNDA: now also U2.16 (SGND), U2.22 (AGND2), U2.23 (AGND1)
- net QUADSPI_CLK: now also U5.58 (PB2)
- net QUADSPI_BK1_IO3: now reaches QSPI.1 (~{HOLD}/IO3)
- net QUADSPI_BK1_IO3: now also U5.101 (PD13)
- net QUADSPI_BK1_IO0: now reaches QSPI.15 (SI/IO0)
- net QUADSPI_BK1_IO0: now also U5.99 (PD11)
- net QUADSPI_BK1_NCS: now reaches QSPI.7 (~{CE})
- net QUADSPI_BK1_NCS: now also U5.110 (PG6)
- net QUADSPI_BK1_IO1: now reaches QSPI.8 (SO/IO1)
- net QUADSPI_BK1_IO1: now also U5.100 (PD12)
- net QUADSPI_BK1_IO2: now reaches QSPI.9 (~{WP}/IO2)
- net QUADSPI_BK1_IO2: now also U5.1 (PE2)
- new net: C31.2, C32.2
- no-connect marks 0 -> 1
Other:
- note added: "Input Stage"
- note added: "Output Stage"
- moved on the sheet: J1, J2, QSPI

Commit message: Update PCM3060
Parts:
- added C33, C35: 100nF, symbol Device:C
- added C34, C36: 10uF, symbol Device:C
Connections:
- net SAI1_FS is gone; now on net SAI1_FS_A: U2.4 (LRCK1), U5.3 (PE4)
- net SAI1_SCK is gone; now on net SAI1_SCK_A: U2.5 (BCK1), U5.4 (PE5)
- net +3V3: now also U2.24 (V_{CC}), U2.7 (V_{DD}), C33.1, C33.2, C34.1, C34.2, C35.1, C36.1
- net GNDA: now also C35.2, C36.2
- net SAI1_MCLK_A: now reaches U5.111 (PG7)
- net SAI1_MCLK_A: now also U2.6 (SCKI1), U2.9 (SCKI2)
- net I2C1_SCL: now reaches U5.167 (PB8)
- net I2C1_SCL: now also U2.1 (MC/SCL/FMT)
- net I2C1_SDA: now reaches U5.168 (PB9)
- net I2C1_SDA: now also U2.2 (MD/SDA/DEMP)
- net SAI1_SD_B: now reaches U5.2 (PE3)
- net SAI1_SD_B: now also U2.3 (DOUT)
- net SAI1_SD_A: now reaches U5.5 (PE6)
- net SAI1_SD_A: now also U2.12 (DIN)
- net SAI1_SCK_A: now reaches U2.10 (BCK2)
- net SAI1_FS_A: now reaches U2.11 (LRCK2)
Other:
- note added: "available GPIO"
- moved on the sheet: SDRAM, U2
